File: Adafruit FONA SIM5320 3G Breakout.brd (EAGLE design)
At the start: 45.7 x 49.5 mm, 45 parts, among them IC1 MIC29302WU, SW3 B3U-1000P-2P-SMD, U1 SIM5320, X6 SIM_LOCKAMPHENOL

Commit message: 最小構成ver1.1.1
Routing:
- net SIMDATA: track 21.0 -> 20.1 mm
Changed lines of the file:
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@@
 <via x="32.512" y="16.002" extent="1-16" drill="0.5"/>
 <via x="34.925" y="16.002" extent="1-16" drill="0.5"/>
-<via x="38.481" y="48.641" extent="1-16" drill="0.5"/>
-<via x="37.084" y="48.768" extent="1-16" drill="0.5"/>
 <contactref element="ANT1" pad="GND2"/>
 <contactref element="ANT1" pad="GND1"/>
@@
 <wire x1="34.417" y1="8.89" x2="34.417" y2="10.414" width="0.254" layer="1"/>
 <wire x1="34.417" y1="10.414" x2="35.456" y2="11.453" width="0.254" layer="1"/>
-<wire x1="35.456" y1="11.453" x2="35.456" y2="12.474690625" width="0.254" layer="1"/>
-<wire x1="35.456" y1="12.474690625" x2="35.456" y2="13.702" width="0.254" layer="1"/>
-<wire x1="35.456" y1="12.474690625" x2="34.919309375" y2="11.938" width="0.254" layer="1"/>
-<wire x1="34.919309375" y1="11.938" x2="27.305" y2="11.938" width="0.254" layer="1"/>
-<wire x1="27.305" y1="11.938" x2="26.67" y2="11.303" width="0.254" layer="1"/>
-<wire x1="26.67" y1="11.303" x2="26.67" y2="10.287" width="0.254" layer="1"/>
+<wire x1="35.456" y1="11.87885625" x2="35.456" y2="11.453" width="0.254" layer="1"/>
+<wire x1="35.456" y1="11.87885625" x2="35.456" y2="13.702" width="0.254" layer="1"/>
+<wire x1="28.956" y1="10.287" x2="31.369" y2="11.938" width="0.254" layer="1"/>
+<wire x1="28.956" y1="10.287" x2="26.67" y2="10.287" width="0.254" layer="1"/>
 <via x="26.67" y="10.287" extent="1-16" drill="0.5"/>
 <wire x1="26.67" y1="10.287" x2="26.67" y2="11.302" width="0.254" layer="16"/>
 <wire x1="26.67" y1="11.302" x2="27.283" y2="11.915" width="0.254" layer="16"/>
+<wire x1="31.369" y1="11.938" x2="35.39685625" y2="11.938" width="0.254" layer="1"/>
+<wire x1="35.39685625" y1="11.938" x2="35.456" y2="11.87885625" width="0.254" layer="1"/>
 </signal>
 <signal name="RI">

Commit message: 最小構成ver1.1.2
Parts:
- moved R5 0.76 mm to (27.1, 47.0)
- moved D3 0.51 mm to (29.2, 46.9)
- moved C2 0.40 mm to (38.5, 47.1)
- moved R4 0.38 mm to (31.2, 46.9)
- moved C9 0.25 mm to (34.9, 46.9)
- moved D4 0.25 mm to (33.0, 46.9)
Routing:
- net UART_DTR: track 37.3 -> 31.4 mm
- net UART_RXD: track 27.6 -> 25.1 mm
- net UART_CTS: track 28.3 -> 26.6 mm
- net RI: track 47.6 -> 46.4 mm
- net NETSTAT: track 49.1 -> 50.0 mm
- net RESET_5V: track 26.5 -> 25.5 mm
- net SIMDATA: track 20.1 -> 19.2 mm

Commit message: 最小構成ver1.1.3
Routing:
- net UART_DTR: track 31.4 -> 31.5 mm, vias 2 -> 1
Changed lines of the file:
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@@
 <signal name="UART_DTR">
 <contactref element="U1" pad="72"/>
-<via x="18.923" y="11.938" extent="1-16" drill="0.5"/>
 <via x="18.923" y="27.178" extent="1-16" drill="0.5"/>
 <wire x1="18.923" y1="27.178" x2="13.98" y2="27.178" width="0.254" layer="1"/>
 <wire x1="13.98" y1="27.178" x2="13.956" y2="27.202" width="0.254" layer="1"/>
 <contactref element="JP1" pad="9"/>
-<wire x1="21.59" y1="1.778" x2="21.59" y2="3.683" width="0.254" layer="1"/>
-<wire x1="21.59" y1="3.683" x2="18.923" y2="6.604" width="0.254" layer="1"/>
-<wire x1="18.923" y1="6.604" x2="18.923" y2="11.938" width="0.254" layer="1"/>
-<wire x1="18.923" y1="27.178" x2="18.923" y2="11.938" width="0.254" layer="16"/>
+<wire x1="18.923" y1="4.445" x2="21.59" y2="1.778" width="0.254" layer="16"/>
+<wire x1="18.923" y1="27.178" x2="18.923" y2="4.445" width="0.254" layer="16"/>
 </signal>
 <signal name="UART_CTS">
@@
 <contactref element="U1" pad="56"/>
 <contactref element="JP2" pad="1"/>
-<wire x1="24.511" y1="48.26" x2="24.257" y2="48.26" width="0.4064" layer="1"/>
-<wire x1="24.257" y1="48.26" x2="23.114" y2="47.117" width="0.4064" layer="1"/>
-<wire x1="23.114" y1="47.117" x2="23.114" y2="44.704" width="0.4064" layer="1"/>
+<wire x1="23.114" y1="44.704" x2="23.114" y2="46.863" width="0.4064" layer="1"/>
 <wire x1="23.114" y1="44.704" x2="23.495" y2="44.323" width="0.4064" layer="1"/>
 <wire x1="23.495" y1="44.323" x2="23.495" y2="43.741" width="0.4064" layer="1"/>
 <wire x1="23.495" y1="43.741" x2="23.456" y2="43.702" width="0.4064" layer="1"/>
+<wire x1="23.114" y1="46.863" x2="24.511" y2="48.26" width="0.4064" layer="1"/>
 </signal>
 <signal name="I2C_SCL">
